File: tutorial1.kicad_pcb (KiCad board)
At the start: 2 copper layers, 25 x 25 mm, 7 parts, among them J1 Conn_01x03_Male, U1 PIC12C508A-ISN

Commit message: #update:実習に伴う更新
Parts:
- added G***: LOGO, LOGO, F.Cu at (153.0, 109.0)
Other:
- board size 25 x 25 mm -> 48.3 x 39.8 mm
