File: tutorial1.kicad_sch (KiCad schematic)
At the start: 6 parts, among them J1 Conn_01x03_Male, U1 PIC12C508A-ISN

Commit message: #make:作業に伴う関連ファイルのアップデート
Parts:
- C1: footprint (none) -> Capacitor_SMD:C_0603_1608Metric_Pad1.08x0.95mm_HandSolder
- D1: footprint (none) -> LED_SMD:LED_0603_1608Metric_Pad1.05x0.95mm_HandSolder
- J1: footprint (none) -> Connector_PinHeader_2.54mm:PinHeader_1x03_P2.54mm_Vertical
- R1, R2: footprint (none) -> Resistor_SMD:R_0603_1608Metric_Pad0.98x0.95mm_HandSolder
- U1: footprint Package_DIP:DIP-8_W7.62mm -> Package_SO:SOIC-8_3.9x4.9mm_P1.27mm
Changed lines of the file:
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@@
       (effects (font (size 1.27 1.27)) (justify left))
     )
-    (property "Footprint" "Package_DIP:DIP-8_W7.62mm" (id 2) (at 195.58 68.58 0)
+    (property "Footprint" "Package_SO:SOIC-8_3.9x4.9mm_P1.27mm" (id 2) (at 195.58 68.58 0)
       (effects (font (size 1.27 1.27)) hide)
     )
@@
     (property "Reference" "C1" (id 0) (at 158.75 53.34 90))
     (property "Value" "0.01u" (id 1) (at 158.75 55.88 90))
-    (property "Footprint" "" (id 2) (at 154.94 61.9252 0)
+    (property "Footprint" "Capacitor_SMD:C_0603_1608Metric_Pad1.08x0.95mm_HandSolder" (id 2) (at 154.94 61.9252 0)
       (effects (font (size 1.27 1.27)) hide)
     )
@@
     (property "Reference" "R1" (id 0) (at 80.01 104.14 90))
     (property "Value" "100" (id 1) (at 80.01 106.68 90))
-    (property "Footprint" "" (id 2) (at 80.01 108.077 90)
+    (property "Footprint" "Resistor_SMD:R_0603_1608Metric_Pad0.98x0.95mm_HandSolder" (id 2) (at 80.01 108.077 90)
       (effects (font (size 1.27 1.27)) hide)
     )
@@
     (property "Reference" "R2" (id 0) (at 229.87 68.58 90))
     (property "Value" "1k" (id 1) (at 229.87 71.12 90))
-    (property "Footprint" "" (id 2) (at 229.87 73.152 90)
+    (property "Footprint" "Resistor_SMD:R_0603_1608Metric_Pad0.98x0.95mm_HandSolder" (id 2) (at 229.87 73.152 90)
       (effects (font (size 1.27 1.27)) hide)
     )
@@
     (property "Reference" "D1" (id 0) (at 214.3125 68.58 0))
     (property "Value" "LED" (id 1) (at 214.3125 71.12 0))
-    (property "Footprint" "" (id 2) (at 215.9 74.93 0)
+    (property "Footprint" "LED_SMD:LED_0603_1608Metric_Pad1.05x0.95mm_HandSolder" (id 2) (at 215.9 74.93 0)
       (effects (font (size 1.27 1.27)) hide)
     )
@@
     (property "Reference" "J1" (id 0) (at 49.53 102.235 0))
     (property "Value" "Conn_01x03_Male" (id 1) (at 49.53 104.775 0))
-    (property "Footprint" "" (id 2) (at 48.895 109.855 0)
+    (property "Footprint" "Connector_PinHeader_2.54mm:PinHeader_1x03_P2.54mm_Vertical" (id 2) (at 48.895 109.855 0)
       (effects (font (size 1.27 1.27)) hide)
     )
@@
     )
     (path "/0cf252ad-8293-46b7-b205-f41e6d9a8697"
-      (reference "C1") (unit 1) (value "0.01u") (footprint "")
+      (reference "C1") (unit 1) (value "0.01u") (footprint "Capacitor_SMD:C_0603_1608Metric_Pad1.08x0.95mm_HandSolder")
     )
     (path "/c6f761ae-aec8-47bd-a15b-96aadd04470f"
-      (reference "D1") (unit 1) (value "LED") (footprint "")
+      (reference "D1") (unit 1) (value "LED") (footprint "LED_SMD:LED_0603_1608Metric_Pad1.05x0.95mm_HandSolder")
     )
     (path "/d847067d-dd58-4d80-8dac-87973e08e134"
-      (reference "J1") (unit 1) (value "Conn_01x03_Male") (footprint "")
+      (reference "J1") (unit 1) (value "Conn_01x03_Male") (footprint "Connector_PinHeader_2.54mm:PinHeader_1x03_P2.54mm_Vertical")
     )
     (path "/74f3c7fe-24ef-4a24-be3b-b7517c07250a"
-      (reference "R1") (unit 1) (value "100") (footprint "")
+      (reference "R1") (unit 1) (value "100") (footprint "Resistor_SMD:R_0603_1608Metric_Pad0.98x0.95mm_HandSolder")
     )
     (path "/b8860185-f4b6-4df9-904a-e9c1bcaac6e5"
-      (reference "R2") (unit 1) (value "1k") (footprint "")
+      (reference "R2") (unit 1) (value "1k") (footprint "Resistor_SMD:R_0603_1608Metric_Pad0.98x0.95mm_HandSolder")
     )
     (path "/0bc82d82-834b-4296-b539-4d801ae1f4e8"
-      (reference "U1") (unit 1) (value "PIC12C508A-ISN") (footprint "Package_DIP:DIP-8_W7.62mm")
-    )
-  )
+      (reference "U1") (unit 1) (value "PIC12C508A-ISN") (footprint "Package_SO:SOIC-8_3.9x4.9mm_P1.27mm")
+    )
+  )

Commit message: #update:実習に伴う更新
Changed lines of the file:
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@@
     (pin "1")
+  )
+  (symbol (lib_id "0-My_Parts:QP-L") (at 242.57 116.84 0) (unit 1)
+    (in_bom yes) (on_board yes) (fields_autoplaced)
+    (property "Reference" "#G?" (id 0) (at 242.57 109.475 0)
+      (effects (font (size 1.27 1.27)) hide)
+    )
+    (property "Value" "QP-L" (id 1) (at 242.57 124.205 0)
+      (effects (font (size 1.27 1.27)) hide)
+    )
+    (property "Footprint" "" (id 2) (at 242.57 116.84 0)
+      (effects (font (size 1.27 1.27)) hide)
+    )
+    (property "Datasheet" "" (id 3) (at 242.57 116.84 0)
+      (effects (font (size 1.27 1.27)) hide)
+    )
   )
   (symbol (lib_id "MCU_Microchip_PIC12:PIC12C508A-ISN") (at 180.34 85.09 0) (unit 1)
@@
       (reference "#FLG02") (unit 1) (value "PWR_FLAG") (footprint "")
     )
+    (path "/05d70fcc-7852-43e3-bcdf-6502a99e0fa0"
+      (reference "#G?") (unit 1) (value "QP-L") (footprint "")
+    )
     (path "/ec6c01f6-558a-4711-be93-ceddddf9e2d4"
